File: schematic/tinyfm-design.kicad_sch (KiCad schematic)
At the start: 1 part

Commit message: feat: draft schematics
Parts:
- added AE1: Antenna, symbol Device:Antenna
- added C1, C2: 0.1μF, symbol Device:C
- added C3: 0.01μF, symbol Device:C
- added C4: 4–40pF, symbol Device:C_Variable
- added C5: 4.7pF, symbol Device:C
- added L1: 0.1μH, symbol Device:L
- added Q1, Q2: 2N3904, symbol Simulation_SPICE:NPN
- added R1, R4, R6: 10kΩ, symbol Device:R
- added R2: 1MΩ, symbol Device:R
- added R3: 100KΩ, symbol Device:R
- added R5: 100Ω, symbol Device:R
- added R7: 1kΩ, symbol Device:R
Connections:
- net Earth: now reaches MIC.1 (-)
- net Earth: now also R3.2, R5.2, R7.2
- net at MIC.2 (+): now also C1.1, R1.2
- new net: C1.2, Q1.2 (B), R2.2, R3.1
- new net: C2.1, Q1.1 (C), R4.2
- new net: Q1.3 (E), R5.1
- new net: AE1.1 (A), C4.2, C5.1, L1.2, Q2.1 (C)
- new net: C5.2, Q2.3 (E), R7.1
- new net: C2.2, C3.2, Q2.2 (B), R6.2
- new net +9V: C3.1, C4.1, L1.1, R1.1, R2.1, R4.1, R6.1
Other:
- moved on the sheet: MIC
